File: _autosave-MeshtasticStick.kicad_sch (KiCad schematic)
At the start: 40 parts, among them J1 Conn_02x05_Odd_Even, J2 Conn_01x04, J4 Conn_01x04, J5 TYPE-C-31-M-12, U1 MDBT50Q-P1MV2, U2 E22-900M30S, U3 MP2338GTL, U4 AP2112K-3.3, U5 MCP73871-2CA, Y1 Crystal

Commit message: ver1
Parts:
- removed U5: MCP73871-2CA, Package_DFN_QFN:QFN-20-1EP_4x4mm_P0.5mm_EP2.5x2.5mm, symbol Battery_Management:MCP73871-2CA
- added BT1: Battery_Cell, Connector_PinHeader_2.54mm:PinHeader_1x02_P2.54mm_Vertical, symbol Device:Battery_Cell
- added C11, C6: 1nF, Capacitor_SMD:C_0201_0603Metric, symbol Device:C
- added C12: 47uF, Capacitor_SMD:CP_Elec_6.3x7.7, symbol Device:C
- added C13: 10nF, Capacitor_SMD:C_0603_1608Metric, symbol Device:C
- added C14: 4.7uF, Capacitor_SMD:C_0603_1608Metric, symbol Device:C
- added C15: 1nF, Capacitor_SMD:C_0603_1608Metric, symbol Device:C
- added C3: 1uF, Capacitor_SMD:C_0201_0603Metric, symbol Device:C
- added C8: 10uF, Capacitor_SMD:C_0201_0603Metric, symbol Device:C
- added D2: SMM4F5.0A, Diode_SMD:D_SMP_DO-220AA, symbol Device:D_TVS_Small
- added J5: Conn_01x02, Connector_PinHeader_2.54mm:PinHeader_1x02_P2.54mm_Vertical, symbol Connector_Generic:Conn_01x02
- added JP2, JP3: Jumper_2_Bridged, Jumper:SolderJumper-2_P1.3mm_Bridged2Bar_RoundedPad1.0x1.5mm, symbol Jumper:Jumper_2_Bridged
- added JP4: Jumper_2_Open, Jumper:SolderJumper-2_P1.3mm_Open_RoundedPad1.0x1.5mm, symbol Jumper:Jumper_2_Open
- added L2: 10uH, Fuse:Fuse_1210_3225Metric, symbol Device:L
- added R10: 2.2M, Capacitor_SMD:C_0603_1608Metric, symbol Device:R
- added R11: 820K, Capacitor_SMD:C_0603_1608Metric, symbol Device:R
- added R14: 3.3K, Capacitor_SMD:C_0603_1608Metric, symbol Device:R
- added R15, R4, R5, R6: 1K, Capacitor_SMD:C_0603_1608Metric, symbol Device:R
- added R16: 24K, Capacitor_SMD:C_0603_1608Metric, symbol Device:R
- added R17, R18, R20, R21, R7: DNM, Capacitor_SMD:C_0603_1608Metric, symbol Device:R
- added R19: 470R, Capacitor_SMD:C_0603_1608Metric, symbol Device:R
- added R8, R9: 0R, Capacitor_SMD:C_0603_1608Metric, symbol Device:R
- added U2: SPV1040T, STMicroelectronics SPV1040T:SOP65P640X120-8N, symbol SPV1040T:SPV1040T
- added U5: L6924D, L6924D footprint:QFN50P300X300X100-17N, symbol L6924D:L6924D
- C10: renamed from C4; footprint (none) -> Capacitor_SMD:C_0603_1608Metric
- C7: renamed from C12; footprint (none) -> Capacitor_SMD:CP_Elec_6.3x7.7
- C9: renamed from C3; footprint (none) -> Capacitor_SMD:C_0603_1608Metric
- D1: footprint (none) -> Diode_SMD:D_SOD-123F
- D3: renamed from D2; footprint (none) -> Diode_SMD:D_SOD-123F
- F1: footprint (none) -> Fuse:Fuse_1210_3225Metric
- J1: renamed from J5; footprint TYPE-C-31-M-12:HRO_TYPE-C-31-M-12 -> TYPE-C-31-M-12 footprint:HRO_TYPE-C-31-M-12
- J2: renamed from J1; footprint (none) -> Connector_PinHeader_1.27mm:PinHeader_2x05_P1.27mm_Vertical
- J3: renamed from J2; footprint (none) -> Connector_PinHeader_2.54mm:PinHeader_1x04_P2.54mm_Vertical
- J4: footprint (none) -> Connector_PinHeader_2.54mm:PinHeader_1x04_P2.54mm_Vertical
- JP1: footprint (none) -> Jumper:SolderJumper-3_P1.3mm_Open_RoundedPad1.0x1.5mm
- L1: footprint (none) -> Inductor_SMD:L_1210_3225Metric
- R22: renamed from R5; footprint Resistor_SMD:R_0603_1608Metric -> Capacitor_SMD:C_0603_1608Metric
- R23: renamed from R6; footprint Resistor_SMD:R_0603_1608Metric -> Capacitor_SMD:C_0603_1608Metric
- R24: renamed from R7; footprint Resistor_SMD:R_0603_1608Metric -> Capacitor_SMD:C_0603_1608Metric
- R25: renamed from R8; footprint Resistor_SMD:R_0603_1608Metric -> Capacitor_SMD:C_0603_1608Metric
- R26: renamed from R9; footprint Resistor_SMD:R_0603_1608Metric -> Capacitor_SMD:C_0603_1608Metric
- R27: renamed from R10; footprint Resistor_SMD:R_0603_1608Metric -> Capacitor_SMD:C_0603_1608Metric
- Y1: footprint (none) -> Crystal:Crystal_SMD_2012-2Pin_2.0x1.2mm
- renumbered C11 to C1, C5 to C16, C6 to C17, C7 to C18, C8 to C19, C13 to C2, C9 to C20, C10 to C21, C1 to C4, C2 to C5, L2 to L3, R11 to R1, R3 to R12, R4 to R13, R1 to R3, U4 to U1, U2 to U3, U1 to U4, U3 to U6
Connections:
- net GND: now also BT1.2 (-), C11.2, C12.2, C13.2, C14.2, C15.2, C6.2, C8.2, D2.2 (A2), JP2.1 (A), JP3.1 (A), R11.1, R14.1, R16.1, R18.1, R19.1, R20.1, R21.1, R7.2, U2.2 (GND), U5.6 (GND)
- new net: JP4.1 (A), R20.2
- new net: JP4.2 (B), R17.2, R21.2, U5.14 (VPRE)
- new net: C15.1, R15.2, U5.12 (VREF)
- new net: R14.2, U5.13 (IEND)
- new net: R16.2, U5.15 (IPRG)
- new net: R17.1, R18.2, U5.16 (IPRE)
- new net: C13.1, U5.5 (TPRG)
- new net: JP2.2 (B), U5.7 (SD)
- new net: JP3.2 (B), U5.9 (VOPRG)
- new net: L2.2, U2.3 (LX)
- new net: R9.1, U2.8 (XSHUT)
- new net Ictrl+: C3.2, R4.1, U2.7 (ICTRL_PLUS)
- new net Ictrl-: C3.1, R5.1, U2.6 (ICTRL_MINUS)
- new net NTC: R15.1, R19.2, U5.8 (TH)
- new net PV+: J5.1 (Pin_1), L2.1, R6.1
- new net PV-: J5.2 (Pin_2)
- new net VBAT: BT1.1 (+), C14.1, U5.10 (VOSNS), U5.11 (VOUT)
- new net VIN_sns: C6.1, R6.2, R7.1, R9.2, U2.1 (MPPT-SET), U5.2 (VINSNS)
- new net VOUT_SPV1040: C12.1, R10.2, R5.2, R8.2, U5.1 (VIN)
- new net Vctrl: C11.1, R10.1, R11.2, U2.5 (VCTRL)
- new net Vrs+: C8.1, D2.1 (A1), R4.2, R8.1, U2.4 (VOUT)
Other:
- moved on the sheet: C1, C16, C17, C18, C19, C2, C20, C21, D1, D3, F1, J1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
