File: MeshtasticStick.kicad_sch (KiCad schematic)
At the start: 36 parts, among them J1 Conn_02x05_Odd_Even, J2 Conn_01x04, J4 Conn_01x04, J5 TYPE-C-31-M-12, U1 MDBT50Q-P1MV2, U2 E22-900M30S, U3 MP2338GTL, U4 AP2112K-3.3, Y1 Crystal

Commit message: ver1
Parts:
- added BT1: Battery_Cell, Connector_PinHeader_2.54mm:PinHeader_1x02_P2.54mm_Vertical, symbol Device:Battery_Cell
- added C12: 100uF, Capacitor_SMD:CP_Elec_6.3x7.7, symbol Device:C
- added C13: 1uF, Capacitor_SMD:C_0603_1608Metric, symbol Device:C
- added C14, C16: 1nF, Capacitor_SMD:C_0201_0603Metric, symbol Device:C
- added C15: 10uF, Capacitor_SMD:C_0201_0603Metric, symbol Device:C
- added C17: 1uF, Capacitor_SMD:C_0201_0603Metric, symbol Device:C
- added C18: 4.7uF, Capacitor_SMD:C_0603_1608Metric, symbol Device:C
- added C19: 47uF, Capacitor_SMD:CP_Elec_6.3x7.7, symbol Device:C
- added C20: 10nF, Capacitor_SMD:C_0603_1608Metric, symbol Device:C
- added C21: 1nF, Capacitor_SMD:C_0603_1608Metric, symbol Device:C
- added D2: MBR120VLSFT1G, Diode_SMD:D_SOD-123F, symbol Device:D_Schottky
- added D3: SMM4F5.0A, Diode_SMD:D_SMP_DO-220AA, symbol Device:D_TVS_Small
- added J3: Conn_01x02, Connector_PinHeader_2.54mm:PinHeader_1x02_P2.54mm_Vertical, symbol Connector_Generic:Conn_01x02
- added JP2, JP3: Jumper_2_Bridged, Jumper:SolderJumper-2_P1.3mm_Bridged2Bar_RoundedPad1.0x1.5mm, symbol Jumper:Jumper_2_Bridged
- added JP4: Jumper_2_Open, Jumper:SolderJumper-2_P1.3mm_Open_RoundedPad1.0x1.5mm, symbol Jumper:Jumper_2_Open
- added L3: 10uH, Fuse:Fuse_1210_3225Metric, symbol Device:L
- added R12, R17, R18, R20: 1K, Capacitor_SMD:C_0603_1608Metric, symbol Device:R
- added R13, R23, R24, R26, R27: DNM, Capacitor_SMD:C_0603_1608Metric, symbol Device:R
- added R14, R19: 0R, Capacitor_SMD:C_0603_1608Metric, symbol Device:R
- added R15: 2.2M, Capacitor_SMD:C_0603_1608Metric, symbol Device:R
- added R16: 820K, Capacitor_SMD:C_0603_1608Metric, symbol Device:R
- added R21: 470R, Capacitor_SMD:C_0603_1608Metric, symbol Device:R
- added R22: 3.3K, Capacitor_SMD:C_0603_1608Metric, symbol Device:R
- added R25: 24K, Capacitor_SMD:C_0603_1608Metric, symbol Device:R
- added U6: SPV1040T, STMicroelectronics SPV1040T:SOP65P640X120-8N, symbol SPV1040T:SPV1040T
- added U7: L6924D, L6924D footprint:QFN50P300X300X100-17N, symbol L6924D:L6924D
- C3, C4: footprint (none) -> Capacitor_SMD:C_0603_1608Metric
- D1: footprint (none) -> Diode_SMD:D_SOD-123F
- F1: footprint (none) -> Fuse:Fuse_1210_3225Metric
- J1: footprint (none) -> Connector_PinHeader_1.27mm:PinHeader_2x05_P1.27mm_Vertical
- J2, J4: footprint (none) -> Connector_PinHeader_2.54mm:PinHeader_1x04_P2.54mm_Vertical
- J5: footprint TYPE-C-31-M-12:HRO_TYPE-C-31-M-12 -> TYPE-C-31-M-12 footprint:HRO_TYPE-C-31-M-12
- JP1: footprint (none) -> Jumper:SolderJumper-3_P1.3mm_Open_RoundedPad1.0x1.5mm
- L1: value L -> 10uH; footprint (none) -> Inductor_SMD:L_1210_3225Metric
- R10, R5, R6, R7, R8, R9: footprint Resistor_SMD:R_0603_1608Metric -> Capacitor_SMD:C_0603_1608Metric
- Y1: footprint (none) -> Crystal:Crystal_SMD_2012-2Pin_2.0x1.2mm
Connections:
- net 5V_OUTPUT: now also U2.10 (VCC), U2.9 (VCC), C12.1, D2.1 (K); no longer C8.1, C9.1, L2.2, R5.2, R9.1
- net 5V_USB: now also C13.1
- net GND: now also U2.1 (GND), U2.11 (GND), U2.12 (GND), U2.2 (GND), U2.20 (GND), U2.22 (GND), U2.3 (GND), U2.4 (GND), U2.5 (GND), BT1.2 (-), C12.2, C13.2, C14.2, C15.2, C16.2, C18.2, C19.2, C20.2, C21.2, D3.2 (A2), JP2.1 (A), JP3.1 (A), R13.2, R16.1, R21.1, R22.1, R23.1, R24.1, R25.1, R27.1, U6.2 (GND), U7.6 (GND)
- net LORA_DIO1: now reaches U2.13 (DIO1)
- net LORA_DIO1: now also U1.9 (P0.03)
- net LORA_DIO2: now reaches U2.14 (BUSY)
- net LORA_DIO2: now also U1.13 (P0.28)
- net LORA_RESET: now reaches U2.15 (~{RST})
- net LORA_RESET: now also U1.10 (P0.29)
- net LORA_MISO: now reaches U2.16 (MISO)
- net LORA_MISO: now also U1.7 (P1.14)
- net LORA_MOSI: now reaches U2.17 (MOSI)
- net LORA_MOSI: now also U1.8 (P1.15)
- net LORA_SCK: now reaches U2.18 (SCK)
- net LORA_SCK: now also U1.6 (P1.13)
- net LORA_CS: now reaches U2.19 (NSS)
- net LORA_CS: now also U1.11 (P0.02)
- net SX126X_RXEN: now reaches U2.6 (RXEN)
- net SX126X_RXEN: now also U1.5 (P1.12)
- net SX126X_TXEN: now reaches U2.7 (TXEN)
- net SX126X_TXEN: now also U2.8 (DIO2)
- new net: JP4.1 (A), R23.2
- new net: JP4.2 (B), R24.2, R26.2, U7.14 (VPRE)
- new net: C21.1, R20.2, U7.12 (VREF)
- new net: R22.2, U7.13 (IEND)
- new net: R25.2, U7.15 (IPRG)
- new net: R26.1, R27.2, U7.16 (IPRE)
- new net: C20.1, U7.5 (TPRG)
- new net: JP2.2 (B), U7.7 (SD)
- new net: JP3.2 (B), U7.9 (VOPRG)
- new net: C8.1, C9.1, D2.2 (A), L2.2, R5.2, R9.1
- new net: L3.2, U6.3 (LX)
- new net: R19.1, U6.8 (XSHUT)
- new net Ictrl+: C17.2, R17.1, U6.7 (ICTRL_PLUS)
- new net Ictrl-: C17.1, R18.1, U6.6 (ICTRL_MINUS)
- new net NTC: R20.1, R21.2, U7.8 (TH)
- new net PV+: J3.1 (Pin_1), L3.1, R12.1
- new net PV-: J3.2 (Pin_2)
- new net VBAT: BT1.1 (+), C18.1, U7.10 (VOSNS), U7.11 (VOUT)
- new net VIN_sns: C14.1, R12.2, R13.1, R19.2, U6.1 (MPPT-SET), U7.2 (VINSNS)
- new net VOUT_SPV1040: C19.1, R14.2, R15.2, R18.2, U7.1 (VIN)
- new net Vctrl: C16.1, R15.1, R16.2, U6.5 (VCTRL)
- new net Vrs+: C15.1, D3.1 (A1), R14.1, R17.2, U6.4 (VOUT)
- no-connect marks 3 -> 4
Other:
- note added: "Low Standby Current: 0.01µA (Typ.) Operation Temperature Range: -40°C to +85°C"
- note added: "Max 6V Vin"
- note added: "Thermal shutdown 150 °C"
- moved on the sheet: C1, C10, C11, C2, C3, C4, C5, C6, C7, C8, C9, D1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

Commit message: update readme.md
Parts:
- renumbered C11 to C1, C4 to C10, C16 to C11, C19 to C12, C20 to C13, C18 to C14, C21 to C15, C5 to C16, C6 to C17, C7 to C18, C8 to C19, C13 to C2, C9 to C20, C10 to C21, C17 to C3, C1 to C4, C2 to C5, C14 to C6, C12 to C7, C15 to C8, C3 to C9, D3 to D2, D2 to D3, J5 to J1, J1 to J2, J2 to J3, J3 to J5, L3 to L2, L2 to L3, R11 to R1, R15 to R10, R16 to R11, R3 to R12, R4 to R13, R22 to R14, R20 to R15, R25 to R16, R26 to R17, R27 to R18, R21 to R19, R23 to R20, R24 to R21, R5 to R22, R6 to R23, R7 to R24, R8 to R25, R9 to R26, R10 to R27, R1 to R3, R17 to R4, R18 to R5, R12 to R6, R13 to R7, R14 to R8, R19 to R9, U4 to U1, U6 to U2, U2 to U3, U1 to U4, U7 to U5, U3 to U6

Commit message: [fix] Fix power supply issue and capacitor packaging, complete initial routing
- Fixed power supply issue to improve stability
- Adjusted certain capacitor packages to meet design requirements
- Completed initial PCB routing
- Corrected OLED signal routing to ensure proper display
Parts:
- added C22: 10uF, Capacitor_SMD:C_0603_1608Metric, symbol Device:C
- added D4, D5: LED, LED_SMD:LED_0603_1608Metric, symbol Device:LED
- added D6: MBR120VLSFT1G, Diode_SMD:D_SOD-123F, symbol Device:D_Schottky
- added J6: Conn_01x04, Connector_PinHeader_2.54mm:PinHeader_1x04_P2.54mm_Vertical, symbol Connector_Generic:Conn_01x04
- added R28, R29: 1K, Resistor_SMD:R_0603_1608Metric, symbol Device:R
- added R30: 0R, Resistor_SMD:R_0603_1608Metric, symbol Device:R
- C11, C3, C8: footprint Capacitor_SMD:C_0201_0603Metric -> Capacitor_SMD:C_0603_1608Metric
- C19, C20: footprint Capacitor_SMD:C_0603_1608Metric -> Capacitor_SMD:C_0805_2012Metric
- C6: value 1nF -> 100nF; footprint Capacitor_SMD:C_0201_0603Metric -> Capacitor_SMD:C_0603_1608Metric
- R1, R10, R11, R12, R13, R14, R15, R16, R17, R18, R19, R2, R20, R21, R22, R23, R24, R25, R26, R27, R3, R4, R5, R6, R7, R9: footprint Capacitor_SMD:C_0603_1608Metric -> Resistor_SMD:R_0603_1608Metric
- R8: value 0R -> 10mR; footprint Capacitor_SMD:C_0603_1608Metric -> Resistor_SMD:R_1210_3225Metric
Connections:
- net 3V3 is gone; now on net VCC: C1.1, C4.1, C5.1, JP1.3 (B), L1.1, U1.5 (VOUT), U4.28 (VDD), U4.30 (VDDH)
- net SYS_VIN is gone; now on net VBAT: C17.1, C18.1, R23.2, U6.2 (VIN)
- net VTref is gone; now on net VCC: J2.1 (Pin_1)
- net 5V_USB: now also C12.1, U5.1 (VIN), D4.2 (A), D5.2 (A), D6.1 (K); no longer C2.1, R1.1, U1.1 (VIN)
- net GND: now also U5.17 (EP), J6.4 (Pin_4)
- net OLED_SCL: now also U4.12 (P0.31)
- net OLED_SDA: now also U4.14 (P0.30)
- net PV+: now also C22.1
- net PV-: now also C22.2
- net VBAT: now also C2.1, R1.1, U1.1 (VIN), R30.2; no longer BT1.1 (+), C14.1, U5.11 (VOUT)
- net VCC: now also J6.3 (Pin_3)
- net at U5.3 (ST2): now also R29.2
- net at U5.4 (ST1): now also R28.2
- net DEBUG_TX: now reaches U4.22 (P0.06)
- net DEBUG_TX: now also J6.2 (Pin_2)
- net DEBUG_RX: now reaches U4.24 (P0.08)
- net DEBUG_RX: now also J6.1 (Pin_1)
- net VOUT_SPV1040 renamed Vrs-
- net Vrs-: now also D6.2 (A); no longer C12.1, U5.1 (VIN)
- new net: BT1.1 (+), C14.1, R30.1, U5.11 (VOUT)
- new net: D5.1 (K), R29.1
- new net: D4.1 (K), R28.1
- no-connect marks 4 -> 34
Other:
- moved on the sheet: C10, C9, J2, J3, J4, J5, JP1, R12, R13, R8, Y1

Commit message: 添加貼片完成照片
Parts:
- R25: value 18K -> 43K
Other:
- note added: "EN > 1.2V"
Changed lines of the file:
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@@
 		)
 	)
+	(text "EN > 1.2V\n"
+		(exclude_from_sim no)
+		(at 33.02 250.444 0)
+		(effects
+			(font
+				(size 1.27 1.27)
+			)
+		)
+	)
 	(text "Low Standby Current: 0.01µA (Typ.)\nOperation Temperature Range: -40°C to +85°C"
 		(exclude_from_sim no)
@@
 			)
 		)
-		(property "Value" "18K"
+		(property "Value" "43K"
 			(at 43.18 258.064 0)
 			(effects
